Commit message: sphere_follower

File: src/sphere_follower/urdf/camera.xacro (robot description, xacro)
@@ -14,5 +14,5 @@
          </clip>
        </camera>
-        <plugin name="light_sensor_plugin" filename="/home/diogo/Documents/ROS_workspaces/challenge-husky/devel/lib/libgazebo_light_sensor_plugin.so">
+        <plugin name="light_sensor_plugin" filename="/home/bir/Documents/workspaces_ros/Projetos/challengeBomb_ws/devel/lib/libgazebo_light_sensor_plugin.so">
           <alwaysOn>true</alwaysOn>
           <updateRate>10</updateRate>
@@ -36,5 +36,5 @@
         <origin rpy="0 0 0" xyz="0 0 0"/>
         <geometry>
-          <mesh filename="package://opencv/meshes/camera.stl"/>
+          <mesh filename="package://cimatec_simulation/meshes/camera.stl"/>
         </geometry>
       </visual>
@@ -42,5 +42,5 @@
         <origin rpy="0 0 0" xyz="0 0 0"/>
         <geometry>
-          <mesh filename="package://opencv/meshes/camera.stl"/>
+          <mesh filename="package://cimatec_simulation/meshes/camera.stl"/>
         </geometry>
       </collision>
