Commit message: rviz launch

File: src/challenge_husky/urdf/attachments.urdf.xacro (robot description, xacro)
@@ -5,5 +5,5 @@
   <xacro:include filename="$(find velodyne_description)/urdf/VLP-16.urdf.xacro"/>
   <VLP-16 parent="vlp_support_link" name="velodyne" topic="/velodyne_points" hz="10" samples="440" gpu="${gpu}">
-    <origin xyz="0 0 0.1" rpy="0 0 0" />
+    <origin xyz="0 0 0.13" rpy="0 0 0" />
   </VLP-16>
   <link name="vlp_support_link">
@@ -53,5 +53,5 @@
       <parent link="top_plate_link" />
       <child link="bowler_link" />
-      <origin xyz="0.2 0 0.01" rpy="0 0 0" />
+      <origin xyz="0 0 0.1" rpy="0 0 0" />
     </joint>
   </robot>

Commit message: support ajustment

File: src/challenge_husky/urdf/attachments.urdf.xacro (robot description, xacro)
@@ -5,5 +5,5 @@
   <xacro:include filename="$(find velodyne_description)/urdf/VLP-16.urdf.xacro"/>
   <VLP-16 parent="vlp_support_link" name="velodyne" topic="/velodyne_points" hz="10" samples="440" gpu="${gpu}">
-    <origin xyz="0 0 0.13" rpy="0 0 0" />
+    <origin xyz="0 0 0.08" rpy="0 0 0" />
   </VLP-16>
   <link name="vlp_support_link">
@@ -11,10 +11,10 @@
       <origin xyz="0.0 0.0 0.0" rpy="0.0 0.0 0.0"/>
       <mass value="0.1"/>
-      <inertia ixx="0.003015625" ixy="0.003015625" ixz="0.0" iyy="0.0" iyz="0.0" izz="0.00003125"/>
+      <inertia ixx="0.0000989583" ixy="0" ixz="0.0" iyy="0.0000989583" iyz="0.0" izz="0.00003125"/>
     </inertial>
     <visual name="">
       <origin xyz="0.0 0.0 0.0" rpy="0.0 0.0 0.0"/>
         <geometry>
-          <cylinder radius="0.05" length="0.2"/>
+          <cylinder radius="0.05" length="0.1"/>
         </geometry>
       <material name="">
@@ -26,10 +26,10 @@
       <origin xyz="0.0 0.0 0.0" rpy="0.0 0.0 0.0"/>
         <geometry>
-          <cylinder radius="0.05" length="0.2"/>
+          <cylinder radius="0.05" length="0.1"/>
         </geometry>
     </collision>
   </link>
   <joint name="vlp_support_joint" type="fixed">
-    <origin xyz="0.0 0.0 0.1" rpy="0.0 0.0 0.0"/>
+    <origin xyz="0.0 0.0 0.05" rpy="0.0 0.0 0.0"/>
     <parent link="top_plate_link"/>
     <child link="vlp_support_link"/>
@@ -53,5 +53,5 @@
       <parent link="top_plate_link" />
       <child link="bowler_link" />
-      <origin xyz="0 0 0.1" rpy="0 0 0" />
+      <origin xyz="0 0 0" rpy="0 0 0" />
     </joint>
   </robot>

Commit message: added A-Loam

File: src/challenge_husky/urdf/attachments.urdf.xacro (robot description, xacro)
@@ -2,7 +2,9 @@
 <robot xmlns:xacro="http://www.ros.org/wiki/xacro" name="example">
   <xacro:arg name="gpu" default="false"/>
+  <xacro:arg name="topic" default="/velodyne_points"/>
   <xacro:property name="gpu" value="$(arg gpu)" />
+  <xacro:property name="topic" value="$(arg topic)" />
   <xacro:include filename="$(find velodyne_description)/urdf/VLP-16.urdf.xacro"/>
-  <VLP-16 parent="vlp_support_link" name="velodyne" topic="/velodyne_points" hz="10" samples="440" gpu="${gpu}">
+  <VLP-16 parent="vlp_support_link" name="velodyne" topic="${topic}" hz="10" samples="440" gpu="${gpu}">
     <origin xyz="0 0 0.08" rpy="0 0 0" />
   </VLP-16>

Commit message: exploration

File: src/challenge_husky/urdf/attachments.urdf.xacro (robot description, xacro)
@@ -6,6 +6,7 @@
   <xacro:property name="topic" value="$(arg topic)" />
   <xacro:include filename="$(find velodyne_description)/urdf/VLP-16.urdf.xacro"/>
+  <xacro:include filename="$(find opencv)/urdf/camera.xacro"/>
   <VLP-16 parent="vlp_support_link" name="velodyne" topic="${topic}" hz="10" samples="440" gpu="${gpu}">
-    <origin xyz="0 0 0.08" rpy="0 0 0" />
+    <origin xyz="0 0 0.05" rpy="0 0 0" />
   </VLP-16>
   <link name="vlp_support_link">
@@ -39,4 +40,5 @@
     <limit lower="0.0" upper="0.0" effort="0.0" velocity="0.0"/>
   </joint>
+<!--
     <link name="bowler_link">
       <visual>
@@ -56,4 +58,11 @@
       <child link="bowler_link" />
       <origin xyz="0 0 0" rpy="0 0 0" />
-    </joint>
+    </joint> -->
+<joint name="base_camera_joint" type="fixed">
+  <origin xyz="0.0 0.0 0.11" rpy="0.0 0.0 0.0"/>
+  <parent link="top_plate_link"/>
+  <child link="base_camera"/>
+  <axis xyz="0.0 0.0 0.0"/>
+  <limit lower="0.0" upper="0.0" effort="0.0" velocity="0.0"/>
+</joint>
   </robot>

Commit message: twist_mux

File: src/challenge_husky/urdf/attachments.urdf.xacro (robot description, xacro)
@@ -60,5 +60,5 @@
     </joint> -->
 <joint name="base_camera_joint" type="fixed">
-  <origin xyz="0.0 0.0 0.11" rpy="0.0 0.0 0.0"/>
+  <origin xyz="0.0 0.0 0.185" rpy="0.0 0.0 0.0"/>
   <parent link="top_plate_link"/>
   <child link="base_camera"/>
